File: HATPlus/LEGHAT+.kicad_pcb (KiCad board)
At the start: 4 copper layers, 65 x 56.5 mm, 25 parts, among them J1 Conn_02x20_Odd_Even, J2 Conn_01x02, J3 Conn_01x08, Q2 CSD18540Q5B, SW1 SW_Push, U4 LTC4373IDD-PBF

Commit message: newnew
Parts:
- D1: value D_Schottky -> D_Schottky_AAK
- J1: moved to B.Cu
- moved Q2 65.8 mm to (-20.0, -9.42), turned to 90 degrees
- moved C3 65.2 mm to (-22.5, -2.00), turned to -90 degrees
- moved C5 59.0 mm to (-13.1, -13.2), turned to 180 degrees
- moved J3 54.5 mm to (19.9, 53.0), turned to 180 degrees
- moved U4 53.3 mm to (-11.5, -8.00), turned to 0 degrees
- moved C4 39.8 mm to (4.20, -9.00), turned to 180 degrees
- moved D1 32.1 mm to (38.0, 42.0), turned to -90 degrees
- moved F1 32.0 mm to (38.0, 46.5), turned to 180 degrees
- moved D2 26.7 mm to (41.9, 36.0), turned to 0 degrees
- moved J2 25.5 mm to (39.0, 53.0)
- moved C2 25.3 mm to (44.0, 21.8), turned to 90 degrees
- moved RV1 24.9 mm to (5.00, 38.5), turned to 0 degrees
- moved R1 23.1 mm to (7.00, 32.8), turned to 90 degrees
- moved C1 14.8 mm to (35.5, 36.5)
- moved PS1 11.1 mm to (31.0, 28.0), turned to -90 degrees
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Connections:
- D1 pad 1: Net-(D1-K) -> Net-(D1-A-Pad1)
- D1 pad 2: Net-(D1-A) -> Net-(D1-A-Pad1)
- D1 pad 3: (no net) -> Net-(D1-K)
- F1 pad 1: Net-(D1-A) -> Net-(D1-A-Pad1)
- J1 pad 17: /HAT_3V3 -> unconnected-(J1-Pin_17-Pad17)
Routing:
- net Net-(U4-INTVCC): track 0.00 -> 23.9 mm
- net Net-(PS1-+VOUT): track 0.00 -> 21.3 mm
- net /HAT_5V0: track 0.00 -> 13.4 mm, vias 0 -> 2
- net Net-(Q2-G): track 0.00 -> 5.83 mm
- net /HAT_GND: vias 0 -> 8
- added copper zone on In1.Cu, net /Bat_Neg
- removed copper zone on B.Cu, net /HAT_GND
- removed copper zone on F.Cu, net /HAT_GND
- removed copper zone on In1.Cu, net /HAT_GND

Commit message: newnewenew
Parts:
- J1: footprint SSM-120-F-DV:SAMTEC_SSM-120-X-DV -> Connector_PinSocket_2.54mm:PinSocket_2x20_P2.54mm_Vertical
- moved Q2 35.7 mm to (8.50, 12.1)
- moved C3 35.6 mm to (7.00, 18.0)
- moved U4 35.4 mm to (13.5, 17.0)
- moved C5 33.5 mm to (12.5, 8.50)
- moved J1 24.2 mm to (8.37, 5.27), turned to -90 degrees
- moved C4 24.1 mm to (17.7, 11.0)
- moved PS1 3.66 mm to (31.0, 31.6)
- moved J2 3.54 mm to (35.5, 52.5)
- moved J3 2.62 mm to (17.3, 52.6)
- moved C1 1.50 mm to (35.5, 35.0)
- moved R1 1.50 mm to (7.00, 34.3), turned to -90 degrees
Routing:
- net Net-(U4-INTVCC): track 23.9 -> 0.00 mm
- net Net-(PS1-+VOUT): track 21.3 -> 0.00 mm
- net /HAT_5V0: track 13.4 -> 0.00 mm, vias 2 -> 0
- net Net-(Q2-G): track 5.83 -> 0.00 mm
- net /HAT_GND: vias 8 -> 0
- net /Bat_Neg: vias 0 -> 13

Commit message: nununununu
nunununu
Parts:
- added C7: C, Capacitor_SMD:C_0603_1608Metric, F.Cu at (13.7, 48.0)
- added C8: C, Capacitor_SMD:C_0603_1608Metric, F.Cu at (16.7, 48.0)
- J3: footprint Connector_JST:JST_GH_BM08B-GHS-TBT_1x08-1MP_P1.25mm_Vertical -> Connector_Molex:Molex_MicroClasp_55932-0810_1x08_P2.00mm_Vertical
- moved J3 2.80 mm to (14.5, 53.0), turned to 0 degrees
- moved J2 1.50 mm to (37.0, 52.5)
Connections:
- net /ENC2_CSn renamed /SPI1_CSn1
- J1 pad 1: unconnected-(J1-Pin_1-Pad1) -> /HAT_3.3V
- J1 pad 12: /ENC1_CSn -> /SPI1_CSn2
- J1 pad 17: unconnected-(J1-Pin_17-Pad17) -> /HAT_3.3V
- J1 pad 36: /DAQ_CSn -> /SPI1_CSn0
- J3 pad 1: unconnected-(J3-Pin_1-Pad1) -> /HAT_3.3V
- J3 pad 2: /DAQ_CSn -> /SPI1_CSn2
- J3 pad 4: /ENC1_CSn -> /SPI1_CSn0
Routing:
- net /HAT_GND: track 0.00 -> 66.7 mm, vias 0 -> 31
- net /HAT_3.3V: track 0.00 -> 55.0 mm
- net /Bat_Neg: track 0.00 -> 41.7 mm, vias 13 -> 12
- net Net-(D1-K): track 0.00 -> 32.8 mm
- net /HAT_5V0: track 0.00 -> 22.8 mm
- net Net-(PS1-+VOUT): track 0.00 -> 15.5 mm
- net Net-(U4-INTVCC): track 0.00 -> 10.4 mm
- net Net-(J2-Pin_1): track 0.00 -> 6.58 mm
- net Net-(D1-A-Pad1): track 0.00 -> 5.67 mm
- net Net-(PS1-TRIM): track 0.00 -> 4.32 mm
- net Net-(Q2-G): track 0.00 -> 2.86 mm
- net Net-(R1-Pad2): track 0.00 -> 2.26 mm
- net Net-(D3-A): track 0.00 -> 1.85 mm
- net Net-(D4-A): track 0.00 -> 1.77 mm

Commit message: almost final
Parts:
- added G***: LOGO, BoardDewsign:logogo, F.Cu at (60.0, 19.5)
- moved R2 17.8 mm to (60.3, 42.6)
- moved D3 17.8 mm to (60.3, 46.1)
- moved R3 17.8 mm to (62.3, 42.7)
- moved D4 17.8 mm to (62.3, 46.1)
- moved C4 9.22 mm to (24.7, 17.0)
- moved C8 7.76 mm to (9.00, 48.8), turned to 90 degrees
- moved C7 6.05 mm to (9.00, 51.8), turned to -90 degrees
- moved C5 3.52 mm to (8.98, 8.50)
- moved Q2 3.04 mm to (11.5, 12.6)
- moved U4 3.00 mm to (16.5, 17.0)
- moved C3 2.03 mm to (9.03, 18.0), turned to 180 degrees
- moved D1 2.02 mm to (40.0, 42.5), turned to 90 degrees
- moved F1 1.80 mm to (39.5, 47.5), turned to 0 degrees
- moved SW1 1.50 mm to (61.0, 33.6)
- moved C1 0.95 mm to (35.5, 36.0)
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Connections:
- F1 pad 2: Net-(J2-Pin_1) -> Net-(J2-Pin_2)
- J2 pad 1: Net-(J2-Pin_1) -> /Bat_Neg
- J2 pad 2: /Bat_Neg -> Net-(J2-Pin_2)
Routing:
- net /SPI1_SCLK: track 0.00 -> 72.4 mm
- net /SPI1_CSn0: track 0.00 -> 66.7 mm
- net /SPI1_MOSI: track 0.00 -> 65.9 mm
- net /GREEN_LED: track 0.00 -> 64.5 mm
- net /SPI1_MISO: track 0.00 -> 62.6 mm
- net /RED_LED: track 0.00 -> 61.3 mm
- net /SPI1_CSn2: track 0.00 -> 52.2 mm
- net /SPI1_CSn1: track 0.00 -> 48.8 mm
- net /USB_Switch: track 0.00 -> 38.2 mm
- net Net-(D1-K): track 32.8 -> 1.64 mm
- net /HAT_GND: track 66.7 -> 39.0 mm, vias 31 -> 24
- net /HAT_5V0: track 22.8 -> 0.00 mm
- net /Bat_Neg: track 41.7 -> 22.9 mm, vias 12 -> 10
- net Net-(PS1-+VOUT): track 15.5 -> 0.00 mm
- net /HAT_3.3V: track 55.0 -> 61.9 mm, vias 0 -> 1
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- added copper zone on F.Cu, net /HAT_5V0
- added copper zone on F.Cu, net Net-(D1-A-Pad1)
- added copper zone on F.Cu, net Net-(D1-K)
- added copper zone on F.Cu, net Net-(PS1-+VOUT)

Commit message: First Draft
Connections:
- J1 pad 12: /SPI1_CSn2 -> /SPI1_CSn0
- J1 pad 36: /SPI1_CSn0 -> /SPI1_CSn2
Routing:
- net /SPI1_CSn2: track 52.2 -> 87.0 mm
- net /SPI1_CSn0: track 66.7 -> 54.4 mm
- net /SPI1_CSn1: track 48.8 -> 51.0 mm
Changed lines of the file:
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@@
 			(layers "*.Cu" "*.Mask")
 			(remove_unused_layers no)
-			(net "/SPI1_CSn2")
+			(net "/SPI1_CSn0")
 			(pinfunction "Pin_12_12")
 			(pintype "passive")
@@
 			(layers "*.Cu" "*.Mask")
 			(remove_unused_layers no)
-			(net "/SPI1_CSn0")
+			(net "/SPI1_CSn2")
 			(pinfunction "Pin_36_36")
 			(pintype "passive")
@@
 	)
 	(segment
+		(start 19.97 2.274365)
+		(end 19.97 5.725635)
+		(width 0.25)
+		(layer "B.Cu")
+		(net "/SPI1_CSn2")
+	)
+	(segment
+		(start 51.55 2.73)
+		(end 50.5 1.68)
+		(width 0.25)
+		(layer "B.Cu")
+		(net "/SPI1_CSn2")
+	)
+	(segment
+		(start 49.515635 1.68)
+		(end 49.465635 1.63)
+		(width 0.25)
+		(layer "B.Cu")
+		(net "/SPI1_CSn2")
+	)
+	(segment
+		(start 20.614365 1.63)
+		(end 19.97 2.274365)
+		(width 0.25)
+		(layer "B.Cu")
+		(net "/SPI1_CSn2")
+	)
+	(segment
+		(start 23 8.755635)
+		(end 23 25.4)
+		(width 0.25)
+		(layer "B.Cu")
+		(net "/SPI1_CSn2")
+	)
+	(segment
+		(start 19.97 5.725635)
+		(end 23 8.755635)
+		(width 0.25)
+		(layer "B.Cu")
+		(net "/SPI1_CSn2")
+	)
+	(segment
+		(start 16.55 52.95)
+		(end 16.5 53)
+		(width 0.15)
+		(layer "B.Cu")
+		(net "/SPI1_CSn2")
+	)
+	(segment
+		(start 16.55 31.85)
+		(end 16.55 52.95)
+		(width 0.25)
+		(layer "B.Cu")
+		(net "/SPI1_CSn2")
+	)
+	(segment
+		(start 23 25.4)
+		(end 16.55 31.85)
+		(width 0.25)
+		(layer "B.Cu")
+		(net "/SPI1_CSn2")
+	)
+	(segment
+		(start 50.5 1.68)
+		(end 49.515635 1.68)
+		(width 0.25)
+		(layer "B.Cu")
+		(net "/SPI1_CSn2")
+	)
+	(segment
+		(start 49.465635 1.63)
+		(end 20.614365 1.63)
+		(width 0.25)
+		(layer "B.Cu")
+		(net "/SPI1_CSn2")
+	)
+	(segment
+		(start 23.75 25.40901)
+		(end 21.75 27.40901)
+		(width 0.25)
+		(layer "B.Cu")
+		(net "/SPI1_CSn1")
+	)
+	(segment
+		(start 23.75 7.95)
+		(end 23.75 25.40901)
+		(width 0.25)
+		(layer "B.Cu")
+		(net "/SPI1_CSn1")
+	)
+	(segment
+		(start 18.5 35.6)
+		(end 18.5 53)
+		(width 0.25)
+		(layer "B.Cu")
+		(net "/SPI1_CSn1")
+	)
+	(segment
+		(start 21.07 5.27)
+		(end 23.75 7.95)
+		(width 0.25)
+		(layer "B.Cu")
+		(net "/SPI1_CSn1")
+	)
+	(segment
+		(start 21.75 27.40901)
+		(end 21.75 32.35)
+		(width 0.25)
+		(layer "B.Cu")
+		(net "/SPI1_CSn1")
+	)
+	(segment
+		(start 21.75 32.35)
+		(end 18.5 35.6)
+		(width 0.25)
+		(layer "B.Cu")
+		(net "/SPI1_CSn1")
+	)
+	(segment
+		(start 24.71 4.814365)
+		(end 24.71 24.97934)
+		(width 0.25)
+		(layer "B.Cu")
+		(net "/SPI1_CSn0")
+	)
+	(segment
+		(start 20.5 34.3)
+		(end 20.5 53)
+		(width 0.25)
+		(layer "B.Cu")
+		(net "/SPI1_CSn0")
+	)
+	(segment
+		(start 24.065635 4.17)
+		(end 24.71 4.814365)
+		(width 0.25)
+		(layer "B.Cu")
+		(net "/SPI1_CSn0")
+	)
+	(segment
 		(start 21.07 2.73)
-		(end 19.97 3.83)
-		(width 0.25)
-		(layer "B.Cu")
-		(net "/SPI1_CSn2")
-	)
-	(segment
-		(start 19.97 23.53)
-		(end 16.5 27)
-		(width 0.25)
-		(layer "B.Cu")
-		(net "/SPI1_CSn2")
-	)
-	(segment
-		(start 19.97 3.83)
-		(end 19.97 23.53)
-		(width 0.25)
-		(layer "B.Cu")
-		(net "/SPI1_CSn2")
-	)
-	(segment
-		(start 16.5 27)
-		(end 16.5 53)
-		(width 0.25)
-		(layer "B.Cu")
-		(net "/SPI1_CSn2")
-	)
-	(segment
-		(start 21.07 23.43)
-		(end 18.5 26)
-		(width 0.25)
-		(layer "B.Cu")
-		(net "/SPI1_CSn1")
-	)
-	(segment
-		(start 21.07 5.27)
-		(end 21.07 23.43)
-		(width 0.25)
-		(layer "B.Cu")
-		(net "/SPI1_CSn1")
-	)
-	(segment
-		(start 18.5 26)
-		(end 18.5 53)
-		(width 0.25)
-		(layer "B.Cu")
-		(net "/SPI1_CSn1")
-	)
-	(segment
-		(start 47.83 4.17)
-		(end 47.57 4.43)
+		(end 22.51 4.17)
 		(width 0.25)
 		(layer "B.Cu")
@@
 	)
 	(segment
-		(start 20.5 29.18934)
-		(end 20.5 53)
+		(start 22.51 4.17)
+		(end 24.065635 4.17)
 		(width 0.25)
 		(layer "B.Cu")
@@
 	)
 	(segment
-		(start 47.57 4.43)
-		(end 47.57 5.93)
+		(start 24.71 24.97934)
+		(end 22.125 27.56434)
 		(width 0.25)
 		(layer "B.Cu")
@@
 	)
 	(segment
-		(start 43.31934 6.37)
-		(end 20.5 29.18934)
+		(start 22.125 27.56434)
+		(end 22.125 32.675)
 		(width 0.25)
 		(layer "B.Cu")
@@
 	)
 	(segment
-		(start 51.55 2.73)
-		(end 50.11 4.17)
-		(width 0.25)
-		(layer "B.Cu")
-		(net "/SPI1_CSn0")
-	)
-	(segment
-		(start 47.57 5.93)
-		(end 47.13 6.37)
-		(width 0.25)
-		(layer "B.Cu")
-		(net "/SPI1_CSn0")
-	)
-	(segment
-		(start 50.11 4.17)
-		(end 47.83 4.17)
-		(width 0.25)
-		(layer "B.Cu")
-		(net "/SPI1_CSn0")
-	)
-	(segment
-		(start 47.13 6.37)
-		(end 43.31934 6.37)
-		(width 0.25)
-		(layer "B.Cu")
+		(start 22.125 32.675)
+		(end 20.5 34.3)
+		(width 0.25)
+		(layer "B.Cu")

Commit message: Draft 2
Connections:
- net /USB_Switch renamed /PWR_Switch
Changed lines of the file:
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@@
 			(size 2.75 1)
 			(layers "F.Cu" "F.Mask" "F.Paste")
-			(net "/USB_Switch")
+			(net "/PWR_Switch")
 			(pinfunction "1_1")
 			(pintype "passive")
@@
 			(size 2.75 1)
 			(layers "F.Cu" "F.Mask" "F.Paste")
-			(net "/USB_Switch")
+			(net "/PWR_Switch")
 			(pinfunction "1_1")
 			(pintype "passive")
@@
 			(layers "*.Cu" "*.Mask")
 			(remove_unused_layers no)
-			(net "/USB_Switch")
+			(net "/PWR_Switch")
 			(pinfunction "Pin_37_37")
 			(pintype "passive")
@@
 	)
 	(segment
-		(start 59 30.74)
-		(end 56.5 28.24)
-		(width 0.25)
-		(layer "F.Cu")
-		(net "/USB_Switch")
-	)
-	(segment
-		(start 54.09 8.09)
-		(end 54.09 5.27)
-		(width 0.25)
-		(layer "F.Cu")
-		(net "/USB_Switch")
-	)
-	(segment
-		(start 55.5 27.24)
-		(end 55.5 9.5)
-		(width 0.25)
-		(layer "F.Cu")
-		(net "/USB_Switch")
-	)
-	(segment
-		(start 55.5 33)
-		(end 55.5 27.24)
-		(width 0.25)
-		(layer "F.Cu")
-		(net "/USB_Switch")
-	)
-	(segment
-		(start 59 36.5)
-		(end 55.5 33)
-		(width 0.25)
-		(layer "F.Cu")
-		(net "/USB_Switch")
-	)
-	(segment
-		(start 55.5 9.5)
-		(end 54.09 8.09)
-		(width 0.25)
-		(layer "F.Cu")
-		(net "/USB_Switch")
-	)
-	(segment
-		(start 56.5 28.24)
-		(end 55.5 27.24)
-		(width 0.25)
-		(layer "F.Cu")
-		(net "/USB_Switch")
-	)
-	(segment
 		(start 10.6975 34.16)
 		(end 7.16 34.16)
@@
 		(net "/RED_LED")
 	)
+	(segment
+		(start 59 30.74)
+		(end 56.5 28.24)
+		(width 0.25)
+		(layer "F.Cu")
+		(net "/PWR_Switch")
+	)
+	(segment
+		(start 54.09 8.09)
+		(end 54.09 5.27)
+		(width 0.25)
+		(layer "F.Cu")
+		(net "/PWR_Switch")
+	)
+	(segment
+		(start 55.5 27.24)
+		(end 55.5 9.5)
+		(width 0.25)
+		(layer "F.Cu")
+		(net "/PWR_Switch")
+	)
+	(segment
+		(start 55.5 33)
+		(end 55.5 27.24)
+		(width 0.25)
+		(layer "F.Cu")
+		(net "/PWR_Switch")
+	)
+	(segment
+		(start 59 36.5)
+		(end 55.5 33)
+		(width 0.25)
+		(layer "F.Cu")
+		(net "/PWR_Switch")
+	)
+	(segment
+		(start 55.5 9.5)
+		(end 54.09 8.09)
+		(width 0.25)
+		(layer "F.Cu")
+		(net "/PWR_Switch")
+	)
+	(segment
+		(start 56.5 28.24)
+		(end 55.5 27.24)
+		(width 0.25)
+		(layer "F.Cu")
+		(net "/PWR_Switch")
+	)
 	(zone

Commit message: thisActuallyTheFinalDraft
Connections:
- J1 pad 17: /HAT_3.3V -> unconnected-(J1-Pin_17-Pad17)
Routing:
- net /HAT_GND: track 39.0 -> 41.0 mm
Changed lines of the file:
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@@
 			(layers "*.Cu" "*.Mask")
 			(remove_unused_layers no)
-			(net "/HAT_3.3V")
+			(net "unconnected-(J1-Pin_17-Pad17)")
 			(pinfunction "Pin_17_17")
-			(pintype "passive")
+			(pintype "passive+no_connect")
 		)
 		(pad "18" thru_hole circle
@@
 	)
 	(gr_text "1"
-		(at 5.842 6.858 0)
+		(at 5.55 7.5 0)
 		(layer "F.SilkS")
 		(effects
@@
 	)
 	(segment
+		(start 9 52.55)
+		(end 9.95 52.55)
+		(width 0.5)
+		(layer "F.Cu")
+		(net "/HAT_GND")
+	)
+	(segment
 		(start 63 30)
 		(end 62 29)
@@
 		(start 18.5042 17.25)
 		(end 19 16.7542)
-		(width 0.5)
+		(width 0.4)
 		(layer "F.Cu")
 		(net "/HAT_GND")
@@
 	)
 	(segment
+		(start 9.95 52.55)
+		(end 10 52.5)
+		(width 0.15)
+		(layer "F.Cu")
+		(net "/HAT_GND")
+	)
+	(segment
 		(start 3.75 39.15)
 		(end 5 40.4)
 		(width 0.25)
+		(layer "F.Cu")
+		(net "/HAT_GND")
+	)
+	(segment
+		(start 9 48)
+		(end 10 48)
+		(width 0.5)
 		(layer "F.Cu")
 		(net "/HAT_GND")
@@
 		(start 17.9478 17.25)
 		(end 18.75 17.25)
-		(width 0.5)
+		(width 0.4)
 		(layer "F.Cu")
 		(net "/HAT_GND")
@@
 	)
 	(segment
+		(start 59 30.74)
+		(end 56.5 28.24)
+		(width 0.25)
+		(layer "F.Cu")
+		(net "/PWR_Switch")
+	)
+	(segment
+		(start 54.09 8.09)
+		(end 54.09 5.27)
+		(width 0.25)
+		(layer "F.Cu")
+		(net "/PWR_Switch")
+	)
+	(segment
+		(start 55.5 27.24)
+		(end 55.5 9.5)
+		(width 0.25)
+		(layer "F.Cu")
+		(net "/PWR_Switch")
+	)
+	(segment
+		(start 55.5 33)
+		(end 55.5 27.24)
+		(width 0.25)
+		(layer "F.Cu")
+		(net "/PWR_Switch")
+	)
+	(segment
+		(start 59 36.5)
+		(end 55.5 33)
+		(width 0.25)
+		(layer "F.Cu")
+		(net "/PWR_Switch")
+	)
+	(segment
+		(start 55.5 9.5)
+		(end 54.09 8.09)
+		(width 0.25)
+		(layer "F.Cu")
+		(net "/PWR_Switch")
+	)
+	(segment
+		(start 56.5 28.24)
+		(end 55.5 27.24)
+		(width 0.25)
+		(layer "F.Cu")
+		(net "/PWR_Switch")
+	)
+	(segment
 		(start 10.6975 34.16)
 		(end 7.16 34.16)
@@
 		(net "/RED_LED")
 	)
-	(segment
-		(start 59 30.74)
-		(end 56.5 28.24)
-		(width 0.25)
-		(layer "F.Cu")
-		(net "/PWR_Switch")
-	)
-	(segment
-		(start 54.09 8.09)
-		(end 54.09 5.27)
-		(width 0.25)
-		(layer "F.Cu")
-		(net "/PWR_Switch")
-	)
-	(segment
-		(start 55.5 27.24)
-		(end 55.5 9.5)
-		(width 0.25)
-		(layer "F.Cu")
-		(net "/PWR_Switch")
-	)
-	(segment
-		(start 55.5 33)
-		(end 55.5 27.24)
-		(width 0.25)
-		(layer "F.Cu")
-		(net "/PWR_Switch")
-	)
-	(segment
-		(start 59 36.5)
-		(end 55.5 33)
-		(width 0.25)
-		(layer "F.Cu")
-		(net "/PWR_Switch")
-	)
-	(segment
-		(start 55.5 9.5)
-		(end 54.09 8.09)
-		(width 0.25)
-		(layer "F.Cu")
-		(net "/PWR_Switch")
-	)
-	(segment
-		(start 56.5 28.24)
-		(end 55.5 27.24)
-		(width 0.25)
-		(layer "F.Cu")
-		(net "/PWR_Switch")
-	)
 	(zone

Commit message: MaybeWeFInallyThere
Parts:
- added TP1: TestPoint, TestPoint:TestPoint_Pad_D1.0mm, F.Cu at (44.7, 48.5)
- added TP2: TestPoint, TestPoint:TestPoint_Pad_D1.0mm, F.Cu at (34.9, 44.2)
- added TP3: TestPoint, TestPoint:TestPoint_Pad_D1.0mm, F.Cu at (35.0, 41.1)
- added TP4: TestPoint, TestPoint:TestPoint_Pad_D1.0mm, F.Cu at (7.55, 14.9)
- added TP5: TestPoint, TestPoint:TestPoint_Pad_D1.0mm, F.Cu at (5.05, 8.55)
- added TP6: TestPoint, TestPoint:TestPoint_Pad_D1.0mm, F.Cu at (9.15, 54.4)
Connections:
- D1 pad 1: Net-(D1-A-Pad1) -> Net-(D1-K)
- D1 pad 2: Net-(D1-A-Pad1) -> Net-(D1-K)
- F1 pad 1: Net-(D1-A-Pad1) -> Net-(D1-K)
Routing:
- net Net-(D1-K): track 1.64 -> 12.3 mm
- net /HAT_5V0: track 0.00 -> 7.90 mm
- net Net-(J2-Pin_2): track 5.50 -> 8.76 mm
- net /HAT_3.3V: track 61.9 -> 65.0 mm
- net Net-(PS1-+VOUT): track 0.00 -> 2.25 mm
- net /HAT_GND: vias 24 -> 25
- net /Bat_Neg: vias 10 -> 11
- removed copper zone on F.Cu, net Net-(D1-A-Pad1)
