File: HATPlus/LEGHAT+.kicad_sch (KiCad schematic)
At the start: 25 parts, among them J1 Conn_02x20_Odd_Even, J2 Conn_01x02, J3 Conn_01x08, Q2 CSD18540Q5B, SW1 SW_Push, U4 LTC4373IDD-PBF

Commit message: newnew
Parts:
- removed D1: D_Schottky, Package_TO_SOT_SMD:TO-277A, symbol Device:D_Schottky
- added D1: D_Schottky_AAK, symbol Device:D_Schottky_AAK
Connections:
- net at C1.1, C2.1, D2.1 (K)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: now also D1.3 (K)
- net at F1.1: now also D1.1 (A), D1.2 (A)
Changed lines of the file:
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@@
 		(color 0 0 0 0)
 	)
+	(junction
+		(at 170.18 22.86)
+		(diameter 0)
+		(color 0 0 0 0)
+	)
+	(junction
+		(at 44.45 24.13)
+		(diameter 0)
+		(color 0 0 0 0)
+	)
 	(no_connect
 		(at 256.54 91.44)
@@
 	(wire
 		(pts
+			(xy 170.18 19.05) (xy 170.18 22.86)
+		)
+		(stroke
+			(width 0)
+			(type default)
+		)
+	)
+	(wire
+		(pts
 			(xy 180.34 49.53) (xy 190.5 49.53)
 		)
@@
 	(wire
 		(pts
-			(xy 162.56 19.05) (xy 162.56 22.86)
-		)
-		(stroke
-			(width 0)
-			(type default)
-		)
-	)
-	(wire
-		(pts
 			(xy 186.69 24.13) (xy 190.5 24.13)
 		)
@@
 	(wire
 		(pts
-			(xy 162.56 39.37) (xy 154.94 39.37)
+			(xy 186.69 22.86) (xy 186.69 13.97)
 		)
 		(stroke
@@
 	(wire
 		(pts
-			(xy 186.69 22.86) (xy 186.69 13.97)
+			(xy 44.45 24.13) (xy 43.18 24.13)
 		)
 		(stroke
@@
 	(wire
 		(pts
-			(xy 52.07 24.13) (xy 53.34 24.13)
-		)
-		(stroke
-			(width 0)
-			(type default)
-		)
-	)
-	(wire
-		(pts
 			(xy 172.72 77.47) (xy 182.88 77.47)
 		)
@@
 	(wire
 		(pts
-			(xy 179.07 19.05) (xy 162.56 19.05)
+			(xy 44.45 24.13) (xy 44.45 26.67)
 		)
 		(stroke
@@
 	(wire
 		(pts
+			(xy 179.07 19.05) (xy 170.18 19.05)
+		)
+		(stroke
+			(width 0)
+			(type default)
+		)
+	)
+	(wire
+		(pts
 			(xy 247.65 34.29) (xy 256.54 34.29)
 		)
@@
 	(wire
 		(pts
-			(xy 43.18 24.13) (xy 44.45 24.13)
+			(xy 44.45 24.13) (xy 45.72 24.13)
 		)
 		(stroke
@@
 	(wire
 		(pts
-			(xy 154.94 27.94) (xy 154.94 39.37)
+			(xy 154.94 27.94) (xy 154.94 44.45)
 		)
 		(stroke
@@
 	(wire
 		(pts
-			(xy 35.56 19.05) (xy 24.13 19.05)
+			(xy 24.13 19.05) (xy 35.56 19.05)
 		)
 		(stroke
@@
 	)
 	(label "HAT_GND"
-		(at 154.94 39.37 0)
+		(at 154.94 44.45 0)
 		(effects
 			(font
@@
 	)
 	(label "HAT_GND"
+		(at 162.56 39.37 0)
+		(effects
+			(font
+				(size 1.27 1.27)
+			)
+			(justify left bottom)
+		)
+	)
+	(label "HAT_GND"
 		(at 193.04 77.47 0)
 		(effects
@@
 	)
 	(symbol
-		(lib_id "Device:D_Schottky")
-		(at 48.26 24.13 180)
-		(unit 1)
-		(body_style 1)
-		(exclude_from_sim no)
-		(in_bom yes)
-		(on_board yes)
-		(in_pos_files yes)
-		(dnp no)
-		(fields_autoplaced yes)
-		(property "Reference" "D1"
-			(at 48.5775 17.78 0)
-			(show_name no)
-			(do_not_autoplace no)
-			(effects
-				(font
-					(size 1.27 1.27)
-				)
-			)
-		)
-		(property "Value" "D_Schottky"
-			(at 48.5775 20.32 0)
-			(show_name no)
-			(do_not_autoplace no)
-			(effects
-				(font
-					(size 1.27 1.27)
-				)
-			)
-		)
-		(property "Footprint" "Package_TO_SOT_SMD:TO-277A"
-			(at 48.26 24.13 0)
-			(hide yes)
-			(show_name no)
-			(do_not_autoplace no)
-			(effects
-				(font
-					(size 1.27 1.27)
-				)
-			)
-		)
-		(property "Datasheet" ""
-			(at 48.26 24.13 0)
-			(hide yes)
-			(show_name no)
-			(do_not_autoplace no)
-			(effects
-				(font
-					(size 1.27 1.27)
-				)
-			)
-		)
-		(property "Description" "Schottky diode"
-			(at 48.26 24.13 0)
-			(hide yes)
-			(show_name no)
-			(do_not_autoplace no)
-			(effects
-				(font
-					(size 1.27 1.27)
-				)
-			)
-		)
-		(pin "1"
-		)
-		(pin "2"
-		)
-		(instances
-			(project "LEGHAT+SCHEMATIC"
-				(path "/4eca0b44-7895-4de1-b60b-9e70a6799560"
-					(reference "D1")
-					(unit 1)
-				)
-			)
-			(project "LEGHAT+"
-				(path "/930e3c40-e68c-46d6-8e4e-88a8be0433a8"
-					(reference "D1")
-					(unit 1)
-				)
-			)
-		)
-	)
-	(symbol
 		(lib_id "Device:C")
 		(at 256.54 30.48 0)
@@
 					(unit 1)
 				)
+			)
+		)
+	)
+	(symbol
+		(lib_id "Device:D_Schottky_AAK")
+		(at 49.53 24.13 180)
+		(unit 1)
+		(body_style 1)
+		(exclude_from_sim no)
+		(in_bom yes)
+		(on_board yes)
+		(in_pos_files yes)
+		(dnp no)
+		(property "Reference" "D1"
+			(at 48.641 17.78 0)
+			(show_name no)
+			(do_not_autoplace no)
+			(effects
+				(font
+					(size 1.27 1.27)
+				)
+			)
+		)
+		(property "Value" "D_Schottky_AAK"
+			(at 52.07 20.32 0)
+			(show_name no)
+			(do_not_autoplace no)
+			(effects
+				(font
+					(size 1.27 1.27)
+				)
+			)
+		)
+		(property "Footprint" ""
+			(at 49.53 24.13 0)
+			(hide yes)
+			(show_name no)
+			(do_not_autoplace no)
+			(effects
+				(font
+					(size 1.27 1.27)
+				)
+			)
+		)
+		(property "Datasheet" ""
+			(at 49.53 24.13 0)
+			(hide yes)
+			(show_name no)
+			(do_not_autoplace no)
+			(effects
+				(font
+					(size 1.27 1.27)
+				)
+			)
+		)
+		(property "Description" "Schottky diode, anode on pins 1 and 2"
+			(at 49.53 24.13 0)
+			(hide yes)
+			(show_name no)
+			(do_not_autoplace no)
+			(effects
+				(font
+					(size 1.27 1.27)
+				)
+			)
+		)
+		(pin "3"
+		)
+		(pin "1"
+		)
+		(pin "2"
+		)
+		(instances
+			(project "LEGHAT+"
+				(path "/930e3c40-e68c-46d6-8e4e-88a8be0433a8"
+					(reference "D1")
+					(unit 1)
+				)

Commit message: newnewenew
Parts:
- J1: footprint SSM-120-F-DV:SAMTEC_SSM-120-X-DV -> Connector_PinSocket_2.54mm:PinSocket_2x20_P2.54mm_Vertical
Changed lines of the file:
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@@
 			)
 		)
-		(property "Footprint" "SSM-120-F-DV:SAMTEC_SSM-120-X-DV"
+		(property "Footprint" "Connector_PinSocket_2.54mm:PinSocket_2x20_P2.54mm_Vertical"
 			(at 248.92 81.28 0)
 			(hide yes)

Commit message: nununununu
nunununu
Parts:
- added C7, C8: C, Capacitor_SMD:C_0603_1608Metric, symbol Device:C
- D1: footprint (none) -> Package_TO_SOT_SMD:TO-277A
- J3: footprint Connector_JST:JST_GH_BM08B-GHS-TBT_1x08-1MP_P1.25mm_Vertical -> Connector_Molex:Molex_MicroClasp_55932-0810_1x08_P2.00mm_Vertical
Connections:
- net HAT_GND: now also C7.2, C8.2
- net HAT_3.3V: now reaches J1.1 (Pin_1)
- net HAT_3.3V: now also J1.17 (Pin_17), J3.1 (Pin_1), C7.1, C8.1
- net DAQ_CSn renamed SPI1_CSn0
- net SPI1_CSn0: now also J3.4 (Pin_4); no longer J3.2 (Pin_2)
- net ENC1_CSn renamed SPI1_CSn2
- net SPI1_CSn2: now also J3.2 (Pin_2); no longer J3.4 (Pin_4)
- net ENC2_CSn renamed SPI1_CSn1
- no-connect marks 24 -> 21

Commit message: almost final
Connections:
- net Bat_Neg: now also J2.1 (Pin_1); no longer J2.2 (Pin_2)
- net at F1.2: now also J2.2 (Pin_2); no longer J2.1 (Pin_1)
Other:
- moved on the sheet: D1, F1, J2
Changed lines of the file:
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@@
 	)
 	(junction
-		(at 44.45 24.13)
+		(at 43.18 24.13)
 		(diameter 0)
 		(color 0 0 0 0)
@@
 	(wire
 		(pts
-			(xy 35.56 24.13) (xy 35.56 19.05)
-		)
-		(stroke
-			(width 0)
-			(type default)
-		)
-	)
-	(wire
-		(pts
 			(xy 170.18 19.05) (xy 170.18 22.86)
 		)
@@
 	(wire
 		(pts
-			(xy 15.24 27.94) (xy 24.13 27.94)
+			(xy 20.32 27.94) (xy 19.05 27.94)
 		)
 		(stroke
@@
 	(wire
 		(pts
+			(xy 34.29 19.05) (xy 34.29 24.13)
+		)
+		(stroke
+			(width 0)
+			(type default)
+		)
+	)
+	(wire
+		(pts
 			(xy 240.03 78.74) (xy 240.03 58.42)
 		)
@@
 	(wire
 		(pts
-			(xy 44.45 24.13) (xy 43.18 24.13)
+			(xy 43.18 24.13) (xy 41.91 24.13)
 		)
 		(stroke
@@
 	(wire
 		(pts
-			(xy 44.45 24.13) (xy 44.45 26.67)
+			(xy 43.18 24.13) (xy 43.18 26.67)
 		)
 		(stroke
@@
 	(wire
 		(pts
+			(xy 52.07 24.13) (xy 53.34 24.13)
+		)
+		(stroke
+			(width 0)
+			(type default)
+		)
+	)
+	(wire
+		(pts
 			(xy 195.58 29.21) (xy 195.58 31.75)
 		)
@@
 	(wire
 		(pts
-			(xy 44.45 24.13) (xy 45.72 24.13)
+			(xy 43.18 24.13) (xy 44.45 24.13)
 		)
 		(stroke
@@
 	(wire
 		(pts
-			(xy 24.13 19.05) (xy 35.56 19.05)
+			(xy 24.13 19.05) (xy 34.29 19.05)
 		)
 		(stroke
@@
 	(wire
 		(pts
+			(xy 19.05 25.4) (xy 24.13 25.4)
+		)
+		(stroke
+			(width 0)
+			(type default)
+		)
+	)
+	(wire
+		(pts
 			(xy 193.04 24.13) (xy 195.58 24.13)
 		)
@@
 	)
 	(label "Bat_Neg"
-		(at 15.24 27.94 0)
+		(at 20.32 27.94 0)
 		(effects
 			(font
@@
 	(symbol
 		(lib_id "Connector_Generic:Conn_01x02")
-		(at 29.21 25.4 0)
+		(at 13.97 27.94 180)
 		(unit 1)
 		(body_style 1)
@@
 		(fields_autoplaced yes)
 		(property "Reference" "J2"
-			(at 31.75 25.3999 0)
+			(at 13.97 19.05 0)
 			(show_name no)
 			(do_not_autoplace no)
@@
 					(size 1.27 1.27)
 				)
-				(justify left)
 			)
 		)
 		(property "Value" "Conn_01x02"
-			(at 31.75 27.9399 0)
+			(at 13.97 21.59 0)
 			(show_name no)
 			(do_not_autoplace no)
@@
 					(size 1.27 1.27)
 				)
-				(justify left)
 			)
 		)
 		(property "Footprint" "Connector_AMASS:AMASS_XT30UPB-F_1x02_P5.0mm_Vertical"
-			(at 29.21 25.4 0)
+			(at 13.97 27.94 0)
 			(hide yes)
 			(show_name no)
@@
 		)
 		(property "Datasheet" ""
-			(at 29.21 25.4 0)
+			(at 13.97 27.94 0)
 			(hide yes)
 			(show_name no)
@@
 		)
 		(property "Description" "Generic connector, single row, 01x02, script generated (kicad-library-utils/schlib/autogen/connector/)"
-			(at 29.21 25.4 0)
+			(at 13.97 27.94 0)
 			(hide yes)
 			(show_name no)
@@
 	(symbol
 		(lib_id "Device:Fuse")
-		(at 39.37 24.13 270)
+		(at 38.1 24.13 270)
 		(unit 1)
 		(body_style 1)
@@
 		(fields_autoplaced yes)
 		(property "Reference" "F1"
-			(at 39.37 17.78 90)
+			(at 38.1 17.78 90)
 			(show_name no)
 			(do_not_autoplace no)
@@
 		)
 		(property "Value" "Fuse"
-			(at 39.37 20.32 90)
+			(at 38.1 20.32 90)
 			(show_name no)
 			(do_not_autoplace no)
@@
 		)
 		(property "Footprint" "belfuse0680L3000-05:FUSC6125X279N"
-			(at 39.37 22.352 90)
+			(at 38.1 22.352 90)
 			(hide yes)
 			(show_name no)
@@
 		)
 		(property "Datasheet" ""
-			(at 39.37 24.13 0)
+			(at 38.1 24.13 0)
 			(hide yes)
 			(show_name no)
@@
 		)
 		(property "Description" "Fuse"
-			(at 39.37 24.13 0)
+			(at 38.1 24.13 0)
 			(hide yes)
 			(show_name no)
@@
 	(symbol
 		(lib_id "Device:D_Schottky_AAK")
-		(at 49.53 24.13 180)
+		(at 48.26 24.13 180)
 		(unit 1)
 		(body_style 1)
@@
 		(dnp no)
 		(property "Reference" "D1"
-			(at 48.641 17.78 0)
+			(at 47.371 17.78 0)
 			(show_name no)
 			(do_not_autoplace no)
@@
 		)
 		(property "Value" "D_Schottky_AAK"
-			(at 52.07 20.32 0)
+			(at 50.8 20.32 0)
 			(show_name no)
 			(do_not_autoplace no)
@@
 		)
 		(property "Footprint" "Package_TO_SOT_SMD:TO-277A"
-			(at 49.53 24.13 0)
+			(at 48.26 24.13 0)
 			(hide yes)
 			(show_name no)
@@
 		)
 		(property "Datasheet" ""
-			(at 49.53 24.13 0)
+			(at 48.26 24.13 0)
 			(hide yes)
 			(show_name no)
@@
 		)
 		(property "Description" "Schottky diode, anode on pins 1 and 2"
-			(at 49.53 24.13 0)
+			(at 48.26 24.13 0)
 			(hide yes)
 			(show_name no)

Commit message: First Draft
Connections:
- net SPI1_CSn0: now also J1.12 (Pin_12); no longer J1.36 (Pin_36)
- net SPI1_CSn2: now also J1.36 (Pin_36); no longer J1.12 (Pin_12)
Other:
- moved on the sheet: C7, C8
Changed lines of the file:
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@@
 	)
 	(junction
-		(at 175.26 46.99)
+		(at 170.18 46.99)
 		(diameter 0)
 		(color 0 0 0 0)
@@
 	(wire
 		(pts
-			(xy 175.26 46.99) (xy 190.5 46.99)
-		)
-		(stroke
-			(width 0)
-			(type default)
-		)
-	)
-	(wire
-		(pts
 			(xy 179.07 29.21) (xy 193.04 29.21)
 		)
@@
 	(wire
 		(pts
-			(xy 167.64 46.99) (xy 175.26 46.99)
+			(xy 162.56 46.99) (xy 190.5 46.99)
 		)
 		(stroke
@@
 		(pts
 			(xy 256.54 58.42) (xy 259.08 58.42)
+		)
+		(stroke
+			(width 0)
+			(type default)
+		)
+	)
+	(wire
+		(pts
+			(xy 162.56 54.61) (xy 153.67 54.61)
 		)
 		(stroke
@@
 	)
 	(label "HAT_GND"
-		(at 167.64 54.61 0)
+		(at 153.67 54.61 0)
 		(effects
 			(font
@@
 	)
 	(label "HAT_GND"
-		(at 175.26 54.61 0)
+		(at 170.18 54.61 0)
 		(effects
 			(font
@@
 		)
 	)
-	(label "SPI1_CSn2"
+	(label "SPI1_CSn0"
 		(at 261.62 71.12 0)
 		(effects
@@
 		)
 	)
-	(label "SPI1_CSn0"
+	(label "SPI1_CSn2"
 		(at 261.62 101.6 0)
 		(effects
@@
 	(symbol
 		(lib_id "Device:C")
-		(at 167.64 50.8 0)
+		(at 162.56 50.8 0)
 		(unit 1)
 		(body_style 1)
@@
 		(fields_autoplaced yes)
 		(property "Reference" "C7"
-			(at 171.45 49.5299 0)
+			(at 166.37 49.5299 0)
 			(show_name no)
 			(do_not_autoplace no)
@@
 		)
 		(property "Value" "C"
-			(at 171.45 52.0699 0)
+			(at 166.37 52.0699 0)
 			(show_name no)
 			(do_not_autoplace no)
@@
 		)
 		(property "Footprint" "Capacitor_SMD:C_0603_1608Metric"
-			(at 168.6052 54.61 0)
+			(at 163.5252 54.61 0)
 			(hide yes)
 			(show_name no)
@@
 		)
 		(property "Datasheet" ""
-			(at 167.64 50.8 0)
+			(at 162.56 50.8 0)
 			(hide yes)
 			(show_name no)
@@
 		)
 		(property "Description" "Unpolarized capacitor"
-			(at 167.64 50.8 0)
+			(at 162.56 50.8 0)
 			(hide yes)
 			(show_name no)
@@
 	(symbol
 		(lib_id "Device:C")
-		(at 175.26 50.8 0)
+		(at 170.18 50.8 0)
 		(unit 1)
 		(body_style 1)
@@
 		(fields_autoplaced yes)
 		(property "Reference" "C8"
-			(at 179.07 49.5299 0)
+			(at 173.99 49.5299 0)
 			(show_name no)
 			(do_not_autoplace no)
@@
 		)
 		(property "Value" "C"
-			(at 179.07 52.0699 0)
+			(at 173.99 52.0699 0)
 			(show_name no)
 			(do_not_autoplace no)
@@
 		)
 		(property "Footprint" "Capacitor_SMD:C_0603_1608Metric"
-			(at 176.2252 54.61 0)
+			(at 171.1452 54.61 0)
 			(hide yes)
 			(show_name no)
@@
 		)
 		(property "Datasheet" ""
-			(at 175.26 50.8 0)
+			(at 170.18 50.8 0)
 			(hide yes)
 			(show_name no)
@@
 		)
 		(property "Description" "Unpolarized capacitor"
-			(at 175.26 50.8 0)
-			(hide yes)
-			(show_name no)
+			(at 170.18 50.8 0)
+			(hide yes)
+			(show_name no)

Commit message: Draft 2
Connections:
- net USB_Switch renamed PWR_Switch
Changed lines of the file:
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@@
 		)
 	)
-	(label "USB_Switch"
+	(label "PWR_Switch"
 		(at 172.72 77.47 0)
 		(effects
@@
 		)
 	)
-	(label "USB_Switch"
+	(label "PWR_Switch"
 		(at 229.87 104.14 0)
 		(effects

Commit message: thisActuallyTheFinalDraft
Connections:
- net HAT_3.3V: no longer J1.17 (Pin_17)
- no-connect marks 21 -> 22
Changed lines of the file:
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@@
 		(color 0 0 0 0)
 	)
-	(junction
-		(at 240.03 58.42)
-		(diameter 0)
-		(color 0 0 0 0)
-	)
 	(no_connect
 		(at 256.54 91.44)
@@
 	)
 	(no_connect
+		(at 240.03 78.74)
+	)
+	(no_connect
 		(at 256.54 76.2)
 	)
@@
 	(wire
 		(pts
-			(xy 240.03 58.42) (xy 243.84 58.42)
+			(xy 229.87 58.42) (xy 243.84 58.42)
 		)
 		(stroke
@@
 	(wire
 		(pts
-			(xy 240.03 78.74) (xy 240.03 58.42)
-		)
-		(stroke
-			(width 0)
-			(type default)
-		)
-	)
-	(wire
-		(pts
 			(xy 180.34 62.23) (xy 190.5 62.23)
 		)
@@
 		)
 		(stroke
-			(width 0)
-			(type default)
-		)
-	)
-	(wire
-		(pts
-			(xy 229.87 58.42) (xy 240.03 58.42)
-		)
-		(stroke

Commit message: MaybeWeFInallyThere
Parts:
- added TP1, TP2, TP3, TP4, TP5, TP6: TestPoint, TestPoint:TestPoint_Pad_D1.0mm, symbol Connector:TestPoint
Connections:
- net HAT_3.3V: now also TP6.1
- net HAT_5V0: now also TP5.1
- net at C3.1, PS1.3 (+VOUT), Q2.1 (S)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: now also TP4.1
- net at C1.1, C2.1, D1.3 (K)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: now also D1.1 (A), D1.2 (A), F1.1, TP2.1, TP3.1
- net at F1.2, J2.2 (Pin_2): now also TP1.1
Other:
- moved on the sheet: D1, F1, J2
